File: pcb/8000a/8000a.kicad_sch (KiCad schematic)
At the start: 12 parts, among them J1 Conn_01x11_Male, U1 LM339, U2 LM339, U3 MSP430G2452IPW14

Commit message: debugging the 8000A
Parts:
- removed R3: 200k, Resistor_SMD:R_0805_2012Metric, symbol Device:R
- added C1, C2: C, Capacitor_SMD:C_0805_2012Metric, symbol Device:C
- added J2: USB_B, Connector_USB:USB_B_Lumberg_2411_02_Horizontal, symbol Connector:USB_B
- added PS1: MEE3S0505SC, Converter_DCDC:Converter_DCDC_Murata_MEE3SxxxxSC_THT, symbol Converter_DCDC:MEE3S0505SC
- R1: value 100k -> 150k; footprint Resistor_SMD:R_0805_2012Metric -> Resistor_THT:R_Axial_DIN0207_L6.3mm_D2.5mm_P10.16mm_Horizontal
- R2: value 100k -> 50k; footprint Resistor_SMD:R_0805_2012Metric -> Resistor_THT:R_Axial_DIN0207_L6.3mm_D2.5mm_P10.16mm_Horizontal
- R3: renamed from R4; footprint Resistor_SMD:R_0805_2012Metric -> Resistor_THT:R_Axial_DIN0207_L6.3mm_D2.5mm_P10.16mm_Horizontal
Connections:
- net +5V: now also C1.1, C2.1
- net GND: now also C1.2, C2.2; no longer R2.2
- net S1: now also U1.11 (+); no longer U1.7 (+)
- net S1': now also U1.13, U3.13 (P2.6/XIN/TA0.1); no longer U1.1, U3.9 (TDO/TDI/SDI/SDA/CAOUT/CA7/A7/P1.7)
- net S4: now also U1.7 (+); no longer U1.11 (+)
- net S4': now also U1.1; no longer U1.13
- net VREF1: now also U1.10 (-); no longer U1.6 (-)
- net VREF2: now also R2.2, U1.6 (-); no longer U1.10 (-)
- net W: now also U2.9 (+); no longer U2.11 (+)
- net W': now also U2.14; no longer U2.13
- net X: now also U2.7 (+); no longer U2.9 (+)
- net X': now also U2.1; no longer U2.14
- net Z: now also U2.11 (+); no longer U2.7 (+)
- net Z': now also U2.13; no longer U2.1
- new net Rx: U3.9 (TDO/TDI/SDI/SDA/CAOUT/CA7/A7/P1.7)
Other:
- moved on the sheet: R3, U1B, U1C, U1E, U2A, U2B, U2C, U2D, U2E

Commit message: put low-pass filter on S'
Parts:
- added C3: 68p, Capacitor_SMD:C_0805_2012Metric, symbol Device:C
- added R4: 15k, Resistor_THT:R_Axial_DIN0207_L6.3mm_D2.5mm_P10.16mm_Horizontal, symbol Device:R
Connections:
- net GND: now also C3.2
- net S': now also C3.1, R4.2; no longer U1.14
- new net: R4.1, U1.14
Changed lines of the file:
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@@
   (junction (at 38.1 156.21) (diameter 0) (color 0 0 0 0)
   )
+  (junction (at 123.19 76.2) (diameter 0) (color 0 0 0 0)
+  )
   (junction (at 82.55 104.14) (diameter 0) (color 0 0 0 0)
   )
@@
     (stroke (width 0) (type default) (color 0 0 0 0))
   )
+  (wire (pts (xy 123.19 76.2) (xy 124.46 76.2))
+    (stroke (width 0) (type default) (color 0 0 0 0))
+  )
   (wire (pts (xy 241.3 62.23) (xy 254 62.23))
     (stroke (width 0) (type default) (color 0 0 0 0))
@@
     (stroke (width 0) (type default) (color 0 0 0 0))
   )
+  (wire (pts (xy 123.19 76.2) (xy 123.19 77.47))
+    (stroke (width 0) (type default) (color 0 0 0 0))
+  )
   (wire (pts (xy 241.3 74.93) (xy 254 74.93))
     (stroke (width 0) (type default) (color 0 0 0 0))
   )
+  (wire (pts (xy 121.92 76.2) (xy 123.19 76.2))
+    (stroke (width 0) (type default) (color 0 0 0 0))
+  )
   (wire (pts (xy 38.1 173.99) (xy 50.8 173.99))
     (stroke (width 0) (type default) (color 0 0 0 0))
@@
     (effects (font (size 1.27 1.27)) (justify left bottom))
   )
-  (label "S'" (at 114.3 76.2 0)
+  (label "S'" (at 124.46 76.2 0)
     (effects (font (size 1.27 1.27)) (justify left bottom))
   )
@@
     (pin "7")
   )
+  (symbol (lib_id "power:GND") (at 123.19 85.09 0) (unit 1)
+    (in_bom yes) (on_board yes) (fields_autoplaced)
+    (property "Reference" "#PWR0105" (id 0) (at 123.19 91.44 0)
+      (effects (font (size 1.27 1.27)) hide)
+    )
+    (property "Value" "GND" (id 1) (at 123.19 90.17 0))
+    (property "Footprint" "" (id 2) (at 123.19 85.09 0)
+      (effects (font (size 1.27 1.27)) hide)
+    )
+    (property "Datasheet" "" (id 3) (at 123.19 85.09 0)
+      (effects (font (size 1.27 1.27)) hide)
+    )
+    (pin "1")
+  )
   (symbol (lib_id "Comparator:LM339") (at 101.6 50.8 0) (unit 3)
     (in_bom yes) (on_board yes) (fields_autoplaced)
@@
     (pin "5")
   )
+  (symbol (lib_id "Device:R") (at 118.11 76.2 90) (unit 1)
+    (in_bom yes) (on_board yes) (fields_autoplaced)
+    (property "Reference" "R4" (id 0) (at 118.11 69.85 90))
+    (property "Value" "15k" (id 1) (at 118.11 72.39 90))
+    (property "Footprint" "Resistor_THT:R_Axial_DIN0207_L6.3mm_D2.5mm_P10.16mm_Horizontal" (id 2) (at 118.11 77.978 90)
+      (effects (font (size 1.27 1.27)) hide)
+    )
+    (property "Datasheet" "~" (id 3) (at 118.11 76.2 0)
+      (effects (font (size 1.27 1.27)) hide)
+    )
+    (pin "1")
+    (pin "2")
+  )
   (symbol (lib_id "Comparator:LM339") (at 40.64 165.1 0) (unit 5)
     (in_bom yes) (on_board yes) (fields_autoplaced)
@@
     )
     (pin "1")
+  )
+  (symbol (lib_id "Device:C") (at 123.19 81.28 0) (unit 1)
+    (in_bom yes) (on_board yes) (fields_autoplaced)
+    (property "Reference" "C3" (id 0) (at 127 80.0099 0)
+      (effects (font (size 1.27 1.27)) (justify left))
+    )
+    (property "Value" "68p" (id 1) (at 127 82.5499 0)
+      (effects (font (size 1.27 1.27)) (justify left))
+    )
+    (property "Footprint" "Capacitor_SMD:C_0805_2012Metric" (id 2) (at 124.1552 85.09 0)
+      (effects (font (size 1.27 1.27)) hide)
+    )
+    (property "Datasheet" "~" (id 3) (at 123.19 81.28 0)
+      (effects (font (size 1.27 1.27)) hide)
+    )
+    (pin "1")
+    (pin "2")
   )
   (symbol (lib_id "Device:C") (at 50.8 165.1 0) (unit 1)
@@
       (reference "#PWR0104") (unit 1) (value "+5V") (footprint "")
     )
+    (path "/3fec1831-49fe-435d-a6eb-ba520e55f450"
+      (reference "#PWR0105") (unit 1) (value "GND") (footprint "")
+    )
     (path "/6c70747c-7398-4d7e-8e06-96138bc42993"
       (reference "#PWR0106") (unit 1) (value "GND") (footprint "")
@@
       (reference "C2") (unit 1) (value "C") (footprint "Capacitor_SMD:C_0805_2012Metric")
     )
+    (path "/a77a459c-1f1d-4583-b823-a54a1c799c78"
+      (reference "C3") (unit 1) (value "68p") (footprint "Capacitor_SMD:C_0805_2012Metric")
+    )
     (path "/7be13a36-eb8e-440f-aaac-2fd6665d9f61"
       (reference "H1") (unit 1) (value "MountingHole") (footprint "MountingHole:MountingHole_3.2mm_M3")
@@
       (reference "R3") (unit 1) (value "100k") (footprint "Resistor_THT:R_Axial_DIN0207_L6.3mm_D2.5mm_P10.16mm_Horizontal")
     )
+    (path "/875404be-e359-458a-af29-1bd3403dd55f"
+      (reference "R4") (unit 1) (value "15k") (footprint "Resistor_THT:R_Axial_DIN0207_L6.3mm_D2.5mm_P10.16mm_Horizontal")
+    )
     (path "/6a8413ac-5ff8-4df9-b89c-e049cf617f69"
