File: pcb/8000a_dou/8000a_dou.kicad_sch (KiCad schematic)
At the start: 17 parts, among them J1 Conn_01x11_Male, J2 USB_B, U1 LM339, U2 LM339, U3 MSP430G2452IPW14

Commit message: rename DOU PCB project
Perhaps further PCBs for the 8000A will be designed or a reproduction of
the original schematic.
Other:
- title: (none) -> 8000A DOU
Changed lines of the file:
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@@
 (kicad_sch (version 20211123) (generator eeschema)
   (paper "A4")
+  (title_block
+    (title "8000A DOU")
+  )
   (junction (at 50.8 156.21) (diameter 0) (color 0 0 0 0)
   )
